File: reference/tutorial.sch (KiCad schematic (older format))
At the start: 30 parts

Commit message: Add annotations
Parts:
- R4: renamed from R?; value R_US -> 10K
- gave numbers to parts that had none: 29
Other:
- note added: "EXTERNAL CONNECTORS"
- note added: "MICROCONTROLLER & CAN"
- note added: "MISC PERIPHERALS"
