File: 2020_keychain_PIC/ee_tut/ee_tut.kicad_pcb (KiCad board)
At the start: 2 copper layers, 41.4 x 37.8 mm, 16 parts, among them J1 Programming_Connector, SW1 SW_Push, SW2 SW_Push, SW3 SW_SPST, U1 PIC16LF15313

Commit message: Adress review comments :good_stuff:
Connections:
- C1 pad 1: +BATT -> +3V0
- J1 pad 2: +BATT -> +3V0
- R3 pad 1: +BATT -> +3V0
- SW1 pad 1: +BATT -> +3V0
- SW2 pad 1: +BATT -> +3V0
- SW3 pad 1: Net-(BT1-Pad1) -> +3V0
- SW3 pad 2: +BATT -> Net-(BT1-Pad1)
- SW3 pad 3: (no net) -> Net-(SW3-Pad3)
- U1 pad 1: +BATT -> +3V0
Routing:
- net Net-(BT1-Pad1): track 57.4 -> 51.6 mm
- net Net-(R2-Pad1): track 25.1 -> 30.2 mm
- net +BATT: track 4.01 -> 0.00 mm
- net +3V0: track 0.00 -> 4.01 mm
- net Net-(R1-Pad1): track 21.3 -> 23.1 mm
- net /~MCLR: track 49.6 -> 50.2 mm
- added copper zone on F.Cu, net +3V0
- removed copper zone on F.Cu, net +BATT
Other:
- outline, holes or cut-outs redrawn
- board text added: "ON<->OFF"
