File: 2020_keychain_PIC/ee_tut/ee_tut.sch (KiCad schematic (older format))
At the start: 15 parts, among them J1 Programming_Connector, SW1 SW_Push, SW2 SW_Push, SW3 SW_SPST, U1 PIC16LF15313

Commit message: Adress review comments :good_stuff:
Parts:
- SW3: symbol Switch:SW_SPST -> Switch:SW_SPDT
Connections:
- net at BT1.1 (+): now also SW3.2 (B); no longer SW3.1 (A)
- net +BATT renamed +3V0
- net +3V0: now also SW3.1 (A); no longer SW3.2 (B)
- no-connect marks 0 -> 1
Other:
- note added: "NOTE: +3V0 line is unregulated! depends on battery voltage"
Changed lines of the file:
@@
 $EndComp
 $Comp
-L Switch:SW_SPST SW3
+L Switch:SW_SPDT SW3
 U 1 1 5F5411AF
 P 8250 2350
@@
 Wire Wire Line
 	4700 2600 5050 2600
-$Comp
-L power:+BATT #PWR07
-U 1 1 5F542868
-P 5050 2450
-F 0 "#PWR07" H 5050 2300 50  0001 C CNN
-F 1 "+BATT" H 5065 2623 50  0000 C CNN
-F 2 "" H 5050 2450 50  0001 C CNN
-F 3 "" H 5050 2450 50  0001 C CNN
-	1    5050 2450
-	1    0    0    -1
-$EndComp
 Wire Wire Line
 	5050 2450 5050 2600
 Connection ~ 5050 2600
-$Comp
-L power:+BATT #PWR09
-U 1 1 5F5429ED
-P 6300 2650
-F 0 "#PWR09" H 6300 2500 50  0001 C CNN
-F 1 "+BATT" H 6315 2823 50  0000 C CNN
-F 2 "" H 6300 2650 50  0001 C CNN
-F 3 "" H 6300 2650 50  0001 C CNN
-	1    6300 2650
-	1    0    0    -1
-$EndComp
 Wire Wire Line
 	6300 2650 6300 2750
@@
 Wire Wire Line
 	7950 2850 7950 2750
-$Comp
-L power:+BATT #PWR015
-U 1 1 5F542D6D
-P 8600 2200
-F 0 "#PWR015" H 8600 2050 50  0001 C CNN
-F 1 "+BATT" H 8615 2373 50  0000 C CNN
-F 2 "" H 8600 2200 50  0001 C CNN
-F 3 "" H 8600 2200 50  0001 C CNN
-	1    8600 2200
-	1    0    0    -1
-$EndComp
-Wire Wire Line
-	8600 2200 8600 2350
-Wire Wire Line
-	8600 2350 8450 2350
+Wire Wire Line
+	8600 2100 8600 2250
+Wire Wire Line
+	8600 2250 8450 2250
 Wire Wire Line
 	4300 3350 4400 3350
@@
 Wire Wire Line
 	4400 3350 5150 3350
-$Comp
-L power:+BATT #PWR01
-U 1 1 5F54436E
-P 3800 3250
-F 0 "#PWR01" H 3800 3100 50  0001 C CNN
-F 1 "+BATT" H 3815 3423 50  0000 C CNN
-F 2 "" H 3800 3250 50  0001 C CNN
-F 3 "" H 3800 3250 50  0001 C CNN
-	1    3800 3250
-	1    0    0    -1
-$EndComp
 Wire Wire Line
 	3800 3250 3800 3350
@@
 	4300 4000 4400 4000
 Connection ~ 4400 4000
-$Comp
-L power:+BATT #PWR02
-U 1 1 5F544C15
-P 3800 3900
-F 0 "#PWR02" H 3800 3750 50  0001 C CNN
-F 1 "+BATT" H 3815 4073 50  0000 C CNN
-F 2 "" H 3800 3900 50  0001 C CNN
-F 3 "" H 3800 3900 50  0001 C CNN
-	1    3800 3900
-	1    0    0    -1
-$EndComp
 Wire Wire Line
 	3800 3900 3800 4000
@@
 	1    0    0    -1
 $EndComp
-$Comp
-L power:+BATT #PWR013
-U 1 1 5F548C38
-P 8550 3100
-F 0 "#PWR013" H 8550 2950 50  0001 C CNN
-F 1 "+BATT" H 8565 3273 50  0000 C CNN
-F 2 "" H 8550 3100 50  0001 C CNN
-F 3 "" H 8550 3100 50  0001 C CNN
-	1    8550 3100
-	1    0    0    -1
-$EndComp
 Text Label 8450 3200 2    50   ~ 0
 ~MCLR
@@
 Text Notes 7250 4150 0    50   ~ 0
 2V Vforward max
+NoConn ~ 8450 2450
+$Comp
+L power:+3V0 #PWR?
+U 1 1 5F5ED148
+P 3800 3250
+F 0 "#PWR?" H 3800 3100 50  0001 C CNN
+F 1 "+3V0" H 3815 3423 50  0000 C CNN
+F 2 "" H 3800 3250 50  0001 C CNN
+F 3 "" H 3800 3250 50  0001 C CNN
+	1    3800 3250
+	1    0    0    -1
+$EndComp
+$Comp
+L power:+3V0 #PWR?
+U 1 1 5F5ED906
+P 3800 3900
+F 0 "#PWR?" H 3800 3750 50  0001 C CNN
+F 1 "+3V0" H 3815 4073 50  0000 C CNN
+F 2 "" H 3800 3900 50  0001 C CNN
+F 3 "" H 3800 3900 50  0001 C CNN
+	1    3800 3900
+	1    0    0    -1
+$EndComp
+$Comp
+L power:+3V0 #PWR?
+U 1 1 5F5EDBD4
+P 5050 2450
+F 0 "#PWR?" H 5050 2300 50  0001 C CNN
+F 1 "+3V0" H 5065 2623 50  0000 C CNN
+F 2 "" H 5050 2450 50  0001 C CNN
+F 3 "" H 5050 2450 50  0001 C CNN
+	1    5050 2450
+	1    0    0    -1
+$EndComp
+$Comp
+L power:+3V0 #PWR?
+U 1 1 5F5EDEA2
+P 6300 2650
+F 0 "#PWR?" H 6300 2500 50  0001 C CNN
+F 1 "+3V0" H 6315 2823 50  0000 C CNN
+F 2 "" H 6300 2650 50  0001 C CNN
+F 3 "" H 6300 2650 50  0001 C CNN
+	1    6300 2650
+	1    0    0    -1
+$EndComp
+$Comp
+L power:+3V0 #PWR?
+U 1 1 5F5EE19B
+P 8600 2100
+F 0 "#PWR?" H 8600 1950 50  0001 C CNN
+F 1 "+3V0" H 8615 2273 50  0000 C CNN
+F 2 "" H 8600 2100 50  0001 C CNN
+F 3 "" H 8600 2100 50  0001 C CNN
+	1    8600 2100
+	1    0    0    -1
+$EndComp
+$Comp
+L power:+3V0 #PWR?
+U 1 1 5F5EE469
+P 8550 3100
+F 0 "#PWR?" H 8550 2950 50  0001 C CNN
+F 1 "+3V0" H 8565 3273 50  0000 C CNN
+F 2 "" H 8550 3100 50  0001 C CNN
+F 3 "" H 8550 3100 50  0001 C CNN
+	1    8550 3100
+	1    0    0    -1
+$EndComp
+Text Notes 7450 1800 0    50   ~ 0
+NOTE: +3V0 line is unregulated! depends on battery voltage
 $EndSCHEMATC
